File: L1IFCape.kicad_pcb (KiCad board)
At the start: 2 copper layers, 86.4 x 54.6 mm, 74 parts, among them J1 RF_Shield_One_Piece, J2 SMA, J3 MMCX, P8 BeagleBone_Black_Header, P9 BeagleBone_Black_Header, U1 24CS256, U2 MAX2769BETI+T, U3 MAX31343ETAY+T, U4 TPS717285DCK, U5 TPS717285DCK, U6 DS90LV012A, X1 SIT5156, X2 QPQ1060

Commit message: Version C3 ready for fabrication
Parts:
- removed U6: DS90LV012A, L1IF:SOT-23-5
- added C36: 100 pF, L1IF:C_0603_1608Metric, F.Cu at (125.0, 70.3)
- added C37: 100 pF, L1IF:C_0603_1608Metric, F.Cu at (138.1, 75.8)
- added C38: 100 pF, L1IF:C_0603_1608Metric, F.Cu at (138.1, 69.4)
- added C39: 100 pF, L1IF:C_0603_1608Metric, F.Cu at (136.1, 67.4)
- added G***: LOGO, L1IF:DeviceState, F.Cu at (137.2, 91.9)
- added QR*****: QR-L1IFCape, L1IF:QR-L1IFCape, F.Cu at (176.9, 85.2)
- added R11: 33, L1IF:R_0603_1608Metric, F.Cu at (146.8, 86.3)
- added R12: 33, L1IF:R_0603_1608Metric, F.Cu at (146.8, 89.3)
- added R18: 33, L1IF:R_0603_1608Metric, F.Cu at (130.6, 64.6)
- added R19: 33, L1IF:R_0603_1608Metric, F.Cu at (130.6, 63.1)
- added R2: 0, L1IF:R_0603_1608Metric, F.Cu at (132.3, 86.4)
- added R20: 33, L1IF:R_0603_1608Metric, F.Cu at (125.0, 66.3)
- added R21: 33, L1IF:R_0603_1608Metric, F.Cu at (125.0, 67.8)
- added R22: 33, L1IF:R_0603_1608Metric, F.Cu at (137.0, 61.2)
- added R3: NL, L1IF:R_0603_1608Metric, F.Cu at (133.8, 86.4)
- added R4: 0, L1IF:R_0603_1608Metric, F.Cu at (135.3, 86.4)
- added R5: 0, L1IF:R_0603_1608Metric, F.Cu at (136.8, 86.4)
- added R6: NL, L1IF:R_0603_1608Metric, F.Cu at (138.3, 86.4)
- added TP5: ~{SHDN}, L1IF:TestPoint_THTPad_D1.5mm_Drill0.7mm, F.Cu at (158.6, 55.4)
- C16: value 10 nF -> 100 pF
- G***: footprint L1IF:Padlock-On -> L1IF:PL-Closed
- G***: footprint L1IF:Padlock-Off -> L1IF:PL-Open
- R10, R8, R9: value 10k -> 33
- R7: value 10k -> 0
- TP1, TP2, TP3: footprint L1IF:TestPoint_Pad_D1.0mm -> L1IF:TestPoint_THTPad_D1.5mm_Drill0.7mm
- moved R7 33.6 mm to (139.8, 86.4), turned to -90 degrees
- moved R9 33.3 mm to (142.8, 86.4), turned to 90 degrees
- moved R8 32.3 mm to (141.3, 86.4), turned to 90 degrees
- moved R10 31.3 mm to (144.3, 86.4), turned to -90 degrees
- moved C8 13.6 mm to (152.1, 58.7), turned to 180 degrees
- moved C29 12.4 mm to (149.7, 60.9)
- moved C4 11.4 mm to (151.2, 63.9), turned to -90 degrees
- moved C5 10.6 mm to (151.2, 75.6)
- moved C7 10.6 mm to (149.7, 75.6)
- moved C30 10.5 mm to (149.7, 72.7)
- moved C2 9.98 mm to (154.6, 60.9)
- moved U5 9.85 mm to (152.1, 72.6)
- moved C3 9.85 mm to (154.5, 72.5)
- moved C9 9.85 mm to (152.1, 70.4)
- moved U4 9.81 mm to (152.1, 60.9)
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- renumbered R2 to R13, R3 to R14, R4 to R15, R5 to R16, R6 to R17
Connections:
- net Net-(D1-K) renamed /Active
- net Net-(D2-K) renamed /Passive
- C16 pad 1: /CLKO -> GND
- C16 pad 2: Net-(U2-CLKOUT) -> /2V85D
- R10 pad 1: Net-(U6-IN-) -> /~{SPICS}
- R10 pad 2: GND -> /SPI0.CS0
- R13 pad 2: /I2C0.SDA -> /SDA.I2C0
- R14 pad 2: /I2C0.SCL -> /SCL.I2C0
- R7 pad 1: +3V3 -> /2V85D
- R7 pad 2: /CLKO -> /SDATA
- R8 pad 1: /CLKO -> /SPI0.SCL
- R8 pad 2: GND -> /SCLK
- R9 pad 1: +3V3 -> /SPI0.SDO
- R9 pad 2: Net-(U6-IN-) -> /SDATA
- U1 pad 1: /I2C0.SCL -> /SCL.I2C0
- U1 pad 3: /I2C0.SDA -> /SDA.I2C0
- U2 pad 10: /SPI0.CS0 -> /~{SPICS}
- U2 pad 17: /SQ1H -> Net-(U2-Q1)
- U2 pad 18: /SQ0H -> Net-(U2-Q0)
- U2 pad 20: /SI0H -> Net-(U2-I0)
- U2 pad 21: /SI1H -> Net-(U2-I1)
- U2 pad 26: GND -> /PGM
- U2 pad 8: /SPI0.SDO -> /SDATA
- U2 pad 9: /SPI0.SCL -> /SCLK
- U3 pad 7: /I2C0.SDA -> /SDA.I2C0
- U3 pad 8: /I2C0.SCL -> /SCL.I2C0
Routing:
- net /2V85D: track 26.0 -> 75.4 mm, vias 2 -> 18
- net /~{SPICS}: track 0.00 -> 38.7 mm, vias 0 -> 2
- net /SDA.I2C0: track 0.00 -> 33.1 mm, vias 0 -> 2
- net /I2C0.SDA: track 41.9 -> 8.82 mm, vias 2 -> 0
- net /PGM: track 0.00 -> 28.0 mm, vias 0 -> 2
- net /BBClk: track 4.49 -> 32.1 mm
- net /I2C0.SCL: track 39.7 -> 14.9 mm, vias 4 -> 0
- net /SCLK: track 0.00 -> 24.2 mm
- net /SDATA: track 0.00 -> 23.9 mm, vias 0 -> 4
- net /CLKO: track 23.5 -> 0.00 mm
- net /SCL.I2C0: track 0.00 -> 23.2 mm
- net +3V3: track 41.6 -> 21.7 mm, vias 0 -> 13
- net /SPI0.CS0: track 31.8 -> 14.1 mm, vias 4 -> 1
- net /SPI0.SCL: track 30.1 -> 13.5 mm, vias 4 -> 0
- net /SPI0.SDO: track 26.3 -> 10.2 mm, vias 4 -> 1
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- added copper zone on In2.Cu, net +3V3
- added copper zone on In2.Cu, net /2V85A
- added copper zone on In2.Cu, net /2V85D
- added copper zone on F.Cu, net GND
- added copper zone on In1.Cu, net GND
- removed copper zone on F.Cu, net +3V3
Other:
- copper layers 2 -> 4
- board text removed: "17 18"
- board text removed: "19 20"
- board text removed: "21 22"
- board text removed: "7 8"
- board text removed: "9 10"

Commit message: Cleaned up for fabrication
Parts:
- moved QR***** 69.4 mm to (113.8, 56.4)
- moved G*** 0.66 mm to (136.6, 91.7)
- renumbered R2 to R1, R1 to R10, R3 to R2, R4 to R3, R5 to R4, R6 to R5, R7 to R6, R8 to R7, R9 to R8, R10 to R9
Other:
- board text added: "PWB: ${PWB_VER} ____________"
- board text added: "RXID:"
- board text removed: "PWB:${PWB_VER} ____________"
