File: L1IFCape.kicad_pcb (KiCad board)
At the start: 4 copper layers, 79.4 x 54.6 mm, 93 parts, among them J1 RF_Shield_One_Piece, J2 SMA, J3 MMCX, P8 BeagleBone_Black_Header, P9 BeagleBone_Black_Header, U1 24CS256, U2 MAX2769BETI+T, U3 MAX31343ETAY+T, U4 TPS717285DCK, U5 TPS717285DCK, X1 SIT5156, X2 QPQ1060

Commit message: Clean up for manufacture of D4
Parts:
- moved G*** 0.83 mm to (150.5, 70.9)
Changed lines of the file:
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@@
 	(footprint "L1IF:L1IFCape-D4_SCH"
 		(layer "F.Cu")
-		(at 150.27 70.13)
+		(at 150.54 70.91)
 		(property "Reference" "G***"
 			(at 0 0 0)
