File: L1IFCape.kicad_sch (KiCad schematic)
At the start: 67 parts, among them J1 RF_Shield_One_Piece, J2 SMA, J3 MMCX, P8 BeagleBone_Black_Header, P9 BeagleBone_Black_Header, U1 24CS256, U2 MAX2769BETI+T, U3 MAX31343ETAY+T, U4 TPS717285DCK, U5 TPS717285DCK, U6 DS90LV012A, X1 SIT5156, X2 QPQ1060

Commit message: Version C3 ready for fabrication
Parts:
- removed C16: 10 nF, L1IF:C_0603_1608Metric, symbol L1IF:Capacitor
- removed R10, R9: 10k, L1IF:R_0603_1608Metric, symbol L1IF:10k_0603
- removed R7, R8: 1k, L1IF:R_0603_1608Metric, symbol L1IF:10k_0603
- removed U6: DS90LV012A, L1IF:SOT-23-5, symbol L1IF:DS90LV012A
- added C16, C36, C37, C38, C39: 100 pF, L1IF:C_0603_1608Metric, symbol L1IF:100nF_0603
- added NT1, NT2: NetTie_2, symbol L1IF:NetTie_2
- added R10, R11, R12, R18, R19, R20, R21, R22, R8, R9: 33, L1IF:R_0603_1608Metric, symbol L1IF:Resistor
- added R2, R4, R5, R7: 0, L1IF:R_0603_1608Metric, symbol L1IF:Resistor
- added R3, R6: NL, L1IF:R_0603_1608Metric, symbol L1IF:Resistor
- added TP5: ~{SHDN}, L1IF:TestPoint_THTPad_D1.5mm_Drill0.7mm, symbol L1IF:TestPoint
- C1: Availability (none) -> In Stock; Check_prices (none) -> https://www.snapeda.com/parts/KW-5R5C334-R/Eaton/view-part/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; Description_1 (none) -> Super Capacitor, Radial, Can, 330mF, 5.5V, 50Ohm, 1kHz, Thr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; MANUFACTURER_NAME (none) -> Eaton; MF (none) -> Eaton; MOUSER_PART_NUMBER (none) -> 504-KW-5R5C334-R; MOUSER_PRICE-STOCK (none) -> https://www.mouser.co.uk/ProductDetail/PowerStor-Eaton/KW-5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; MP KR-5R5C105-R -> KW-5R5C334-R; Price (none) -> None
- TP1, TP2, TP3: footprint L1IF:TestPoint_Pad_D1.0mm -> L1IF:TestPoint_THTPad_D1.5mm_Drill0.7mm
- renumbered R2 to R13, R3 to R14, R4 to R15, R5 to R16, R6 to R17
Connections:
- net +1V8: now also NT2.2
- net 2V85A: now also C36.1, C37.1, C38.2
- net 2V85D: now also C16.2, C39.2, R2.1, R6.1, R7.1
- net BBClk: now also R22.2, TP5.1
- net GND: now also C16.1, C36.2, C37.2, C38.1, C39.1, R3.2, R4.1, R5.1; no longer U2.26 (PGM)
- net I2C0.SCL: now also R11.2; no longer R14.2, U1.1 (SCL), U3.8 (SCL)
- net I2C0.SDA: now also R12.1; no longer R13.2, U1.3 (SDA), U3.7 (SDA)
- net SI0H: now also R20.1; no longer U2.20 (I0)
- net SI1H: now also R21.2; no longer U2.21 (I1)
- net SPI0.CS0: now also R10.2; no longer U2.10 (~{CS})
- net SPI0.SCL: now also R8.1; no longer U2.9 (SCLK)
- net SPI0.SDO: now also R9.1; no longer U2.8 (SDATA)
- net SQ0H: now also R18.2; no longer U2.18 (Q0)
- net SQ1H: now also R19.2; no longer U2.17 (Q1)
- net VBUS: now also NT1.2
- net Active: now reaches C11.2, D1.1 (K), J2.1 (In), L1.2
- net at U2.16 (CLKOUT): now also R22.1
- net Passive: now reaches C10.2, D2.1 (K), J3.1 (In)
- new net: R20.2, U2.20 (I0)
- new net: R18.1, U2.18 (Q0)
- new net: R19.1, U2.17 (Q1)
- new net: R21.1, U2.21 (I1)
- new net PGM: R2.2, R3.1, U2.26 (PGM)
- new net SCL.I2C0: R11.1, R14.2, U1.1 (SCL), U3.8 (SCL)
- new net SCLK: R5.2, R6.2, R8.2, U2.9 (SCLK)
- new net SDA.I2C0: R12.2, R13.2, U1.3 (SDA), U3.7 (SDA)
- new net SDATA: R7.2, R9.2, U2.8 (SDATA)
- new net SYS_5V: NT1.1
- new net VADC: NT2.1
- new net ~{SPICS}: R10.1, R4.2, U2.10 (~{CS})
- no-connect marks 64 -> 66
Other:
- note added: "R2 R3 R4 R5 R6 R7 R8 R9 R10 #1 0 NL 0 0 NL 0 NL NL NL Device State 2 #2 0 NL 0 NL 0 0 NL NL NL Device State 6 #3 NL 0 NL NL NL NL 33 33 33 Serial Interface"
- moved on the sheet: C17, C18, P8, R1, TP1, TP2, TP3, TP4

Commit message: Cleaned up for fabrication
Parts:
- renumbered R2 to R1, R1 to R10, R3 to R2, R4 to R3, R5 to R4, R6 to R5, R7 to R6, R8 to R7, R9 to R8, R10 to R9
Other:
- note added: "R1 R2 R3 R4 R5 R6 R7 R8 R9 #1 0 NL 0 0 NL 0 NL NL NL Device State 2 #2 0 NL 0 NL 0 0 NL NL NL Device State 6 #3 NL 0 NL NL NL NL 33 33 33 Serial Interface"
- note removed: "R2 R3 R4 R5 R6 R7 R8 R9 R10 #1 0 NL 0 0 NL 0 NL NL NL Device State 2 #2 0 NL 0 NL 0 0 NL NL NL Device State 6 #3 NL 0 NL NL NL NL 33 33 33 Serial Interface"
Changed lines of the file:
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@@
 	(title_block
 		(title "L1IFCape")
-		(date "2026-08-14")
+		(date "2026-08-15")
 		(rev "${SCH_VER}")
 		(comment 1 "https://cern.ch/cern-ohl ")
@@
 		)
 	)
-	(text "   R2  R3  R4  R5  R6  R7  R8  R9  R10\n#1  0  NL   0   0  NL   0  NL  NL  NL   Device State 2\n#2  0  NL   0  NL   0   0  NL  NL  NL   Device State 6\n#3 NL   0  NL  NL  NL  NL  33  33  33   Serial Interface"
+	(text "   R1  R2  R3  R4  R5  R6  R7  R8  R9\n#1  0  NL   0   0  NL   0  NL  NL  NL   Device State 2\n#2  0  NL   0  NL   0   0  NL  NL  NL   Device State 6\n#3 NL   0  NL  NL  NL  NL  33  33  33   Serial Interface"
 		(exclude_from_sim no)
 		(at 14.732 201.93 0)
 		(effects
 			(font
+				(face "osifont")
 				(size 1.27 1.27)
 			)
@@
 		(in_pos_files yes)
 		(dnp no)
-		(property "Reference" "R2"
+		(property "Reference" "R1"
 			(at 62.484 167.132 0)
 			(show_name no)
@@
 			(project "L1IFCape"
 				(path "/e63e39d7-6ac0-4ffd-8aa3-1841a4541b55"
-					(reference "R2")
+					(reference "R1")
 					(unit 1)
 				)
@@
 		(in_pos_files yes)
 		(dnp no)
-		(property "Reference" "R5"
+		(property "Reference" "R4"
 			(at 68.58 180.086 0)
 			(show_name no)
@@
 			(project "L1IFCape"
 				(path "/e63e39d7-6ac0-4ffd-8aa3-1841a4541b55"
-					(reference "R5")
+					(reference "R4")
 					(unit 1)
 				)
@@
 		(in_pos_files yes)
 		(dnp no)
-		(property "Reference" "R9"
+		(property "Reference" "R8"
 			(at 92.456 45.974 90)
 			(show_name no)
@@
 			(project "L1IFCape"
 				(path "/e63e39d7-6ac0-4ffd-8aa3-1841a4541b55"
-					(reference "R9")
+					(reference "R8")
 					(unit 1)
 				)
@@
 		(in_pos_files yes)
 		(dnp no)
-		(property "Reference" "R1"
+		(property "Reference" "R10"
 			(at 168.656 135.382 90)
 			(show_name no)
@@
 			(project "L1IFCape"
 				(path "/e63e39d7-6ac0-4ffd-8aa3-1841a4541b55"
-					(reference "R1")
+					(reference "R10")
 					(unit 1)
 				)
@@
 		(in_pos_files yes)
 		(dnp no)
-		(property "Reference" "R8"
+		(property "Reference" "R7"
 			(at 96.012 56.896 90)
 			(show_name no)
@@
 			(project "L1IFCape"
 				(path "/e63e39d7-6ac0-4ffd-8aa3-1841a4541b55"
-					(reference "R8")
+					(reference "R7")
 					(unit 1)
 				)
@@
 		(in_pos_files yes)
 		(dnp no)
-		(property "Reference" "R7"
+		(property "Reference" "R6"
 			(at 75.438 166.878 0)
 			(show_name no)
@@
 			(project "L1IFCape"
 				(path "/e63e39d7-6ac0-4ffd-8aa3-1841a4541b55"
-					(reference "R7")
+					(reference "R6")
 					(unit 1)
 				)
@@
 		(in_pos_files yes)
 		(dnp no)
-		(property "Reference" "R3"
+		(property "Reference" "R2"
 			(at 61.214 180.34 0)
 			(show_name no)
@@
 			(project "L1IFCape"
 				(path "/e63e39d7-6ac0-4ffd-8aa3-1841a4541b55"
-					(reference "R3")
+					(reference "R2")
 					(unit 1)
 				)
@@
 		(in_pos_files yes)
 		(dnp no)
-		(property "Reference" "R10"
+		(property "Reference" "R9"
 			(at 34.798 44.704 90)
 			(show_name no)
@@
 			(project "L1IFCape"
 				(path "/e63e39d7-6ac0-4ffd-8aa3-1841a4541b55"
-					(reference "R10")
+					(reference "R9")
 					(unit 1)
 				)
@@
 		(in_pos_files yes)
 		(dnp no)
-		(property "Reference" "R4"
+		(property "Reference" "R3"
 			(at 74.93 179.832 0)
 			(show_name no)
@@
 			(project "L1IFCape"
 				(path "/e63e39d7-6ac0-4ffd-8aa3-1841a4541b55"
-					(reference "R4")
+					(reference "R3")
 					(unit 1)
 				)
@@
 		(in_pos_files yes)
 		(dnp no)
-		(property "Reference" "R6"
+		(property "Reference" "R5"
 			(at 69.088 166.878 0)
 			(show_name no)
@@
 			(project "L1IFCape"
 				(path "/e63e39d7-6ac0-4ffd-8aa3-1841a4541b55"
-					(reference "R6")
+					(reference "R5")
 					(unit 1)
 				)

Commit message: Creating BOM
Parts:
- C10, C11, C18: VPN (none) -> 490-GCM1885C2A471FA16DCT-ND
- C13, C21, C22, C23, C24, C25, C26, C4, C5: VPN (none) -> 399-6856-1-ND
- C14, C8, C9: VPN (none) -> 399-C0603C103F3GECAUTOCT-ND
- C15, C2, C27, C28, C3, C35, C6, C7: VPN (none) -> 490-5241-1-ND
- C17: VPN (none) -> 399-C0603C270F3HACAUTOCT-ND
- C19: value NL -> 470 pF; now not fitted
- C29, C30: value NL -> 10 nF; now not fitted
- C31, C33: VPN (none) -> 399-15708-1-ND
- C32, C34: VPN (none) -> 399-C0805C104K8RACTUCT-ND
- FB1, FB2: VPN (none) -> 490-14399-1-ND
- J1: VPN (none) -> 903-1008-1-ND
- J2: VPN (none) -> ARF1206-ND
- J3: VPN (none) -> ARF1904-ND
- P8, P9: VPN (none) -> 612-SSQ-123-23-G-D-ND
- R1, R3, R4, R6: MFR (none) -> Panasonic; MPN (none) -> ERJ-3GEY0R00V; VPN (none) -> P0.0GCT-ND; Vendor (none) -> DigiKey; Vendor PN (none) -> P0.0GCT-ND
- R10: MFR (none) -> Panasonic; VPN (none) -> P20.0KHCT-ND
- R11, R12, R18, R19, R20, R21, R22, R7, R8, R9: MFR (none) -> Panasonic; MPN (none) -> ERJ-3EKF33R0V; VPN (none) -> P33.0HCT-ND; Vendor (none) -> Digikey
- R17: VPN (none) -> P10.0KHCT-ND
- R2, R5: DNP (none) -> 0; MFR (none) -> Panasonic; MPN (none) -> ERJ-3GEY0R00V; VPN (none) -> P0.0GCT-ND; Vendor (none) -> DigiKey; Vendor PN (none) -> P0.0GCT-ND
- TP5: value ~{SHDN} -> BBClk
